File: pcb/pcbcalc/miyocalc40.kicad_pcb (KiCad board)
At the start: 2 copper layers, 127.7 x 81.4 mm, 57 parts, among them U1 AVR128DA28

Commit message: Multiple updates for rev 1.0
Routing:
- net /colJ: track 126.4 -> 125.4 mm
- net /colG: track 89.8 -> 88.9 mm
- net /colH: track 99.3 -> 98.5 mm
- net /colA: track 92.3 -> 91.5 mm
- net /colI: track 116.9 -> 116.2 mm
- net +3V3: track 106.2 -> 105.5 mm
- net /colD: track 79.6 -> 78.9 mm
- net /colF: track 83.2 -> 82.5 mm
- net /colB: track 84.1 -> 83.5 mm
- net /colC: track 80.2 -> 79.5 mm
- net /colE: track 79.3 -> 78.7 mm
Other:
- board text added: "+"
- board text added: "-"
- board text added: "1"
- board text added: "14"
- board text added: "15"
- board text added: "28"
- board text added: "9"
- board text added: "AVR128DA28"
- board text added: "C1"
- board text added: "C2"
- board text added: "C3"
- board text added: "JLCJLCJLCJLC"
- board text added: "R1"
- board text added: "R2"
- board text added: "Reset"
- board text added: "Rev 1.0"
- board text added: "UPDI"
- board text added: "col A"
- board text added: "col J"
- board text added: "https://github.com/JonathanFerron/MiyoCalc40"
- board text added: "row 1"
- board text added: "row 4"
